File: KiCad_Files/STM32 VGA.kicad_pcb (KiCad board)
At the start: 2 copper layers, 32.8 x 59.9 mm, 35 parts, among them J1 USB_C_Receptacle_USB2.0_16P, J2 DE15_Socket_HighDensity_Mount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, J3 Conn_01x17_Pin, J4 Conn_01x17_Pin, U1 STM32F103C8Tx, U2 AMS1117-3.3, Y1 Crystal_GND24

Commit message: Updated to V1.2 Schematics and PCB
Parts:
- removed the G*** at (203.7, 64.8)
- removed the G*** at (190.1, 65.2)
- removed JP1: SolderJumper_2_Open, Jumper:SolderJumper-2_P1.3mm_Open_RoundedPad1.0x1.5mm
- added BOOT: SKRPACE010, My Footprint Library:SW_SKRPACE010, F.Cu at (201.8, 70.8)
- added RST: SKRPACE010, My Footprint Library:SW_SKRPACE010, F.Cu at (201.8, 66.9)
- moved D1 3.94 mm to (195.3, 73.5)
- moved D2 3.93 mm to (195.3, 75.2)
- moved R10 3.90 mm to (197.0, 64.8)
- moved R11 3.90 mm to (195.0, 64.8)
- moved R7 3.90 mm to (193.0, 64.8)
- moved R8 3.90 mm to (191.0, 64.8)
- moved R9 3.90 mm to (189.0, 64.8)
- moved R12 3.62 mm to (198.8, 73.5)
- moved R13 3.61 mm to (198.8, 75.2)
Routing:
- net Net-(U1-BOOT0): track 4.10 -> 46.9 mm, vias 0 -> 4
- net Net-(J2-Pad13): track 26.6 -> 0.00 mm
- net Net-(J2-Pad14): track 20.4 -> 0.00 mm
- net Net-(U1-NRST): track 17.2 -> 36.7 mm, vias 2 -> 4
- net +3V3: track 128.7 -> 144.8 mm
- net Net-(J2-Pad3): track 9.30 -> 0.00 mm
- net Net-(J2-Pad1): track 9.28 -> 0.00 mm
- net Net-(J2-Pad2): track 8.59 -> 0.00 mm
- net Net-(J4-Pin_1): track 32.7 -> 36.4 mm
- net VSync: track 32.8 -> 36.3 mm
- net GND: track 63.2 -> 60.1 mm, vias 38 -> 34
- net Net-(J4-Pin_2): track 32.0 -> 35.0 mm
- net R: track 27.6 -> 30.2 mm
- net HSync: track 25.0 -> 27.6 mm
- net G: track 29.5 -> 32.0 mm
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Other:
- board text added: "Rev 1.2A 1/1/26"
- board text removed: "Rev 1.1A 11/23/25"
