File: KiCad_Files/STM32 VGA.kicad_sch (KiCad schematic)
At the start: 31 parts, among them J1 USB_C_Receptacle_USB2.0_16P, J2 DE15_Socket_HighDensity_Mount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, J3 Conn_01x17_Pin, J4 Conn_01x17_Pin, U1 STM32F103C8Tx, U2 AMS1117-3.3, Y1 Crystal_GND24

Commit message: Updated to V1.2 Schematics and PCB
Parts:
- removed JP1: SolderJumper_2_Open, Jumper:SolderJumper-2_P1.3mm_Open_RoundedPad1.0x1.5mm, symbol Jumper:SolderJumper_2_Open
- added S1, S2: SKRPACE010, My Footprint Library:SW_SKRPACE010, symbol SKRPACE010:SKRPACE010
- C5, C6: value 10u -> 10pf
Connections:
- net +3V3: now also S2.1, S2.2
- net GND: now also S1.3, S1.4
- net at R5.1, U1.7 (NRST): now also S1.1, S1.2
- net at R6.1, U1.44 (BOOT0): now also S2.3, S2.4
Other:
- moved on the sheet: R5, R6
